File: lpc812-breakout.sch (KiCad schematic (older format))
At the start: 27 parts, among them J1 SWD, J2 Left, J3 Right, Q1 BC847BDW1, SW1 Reset, U1 LPC812M101JDH20, Y1 8MHz

Commit message: Schematic cleanup
Parts:
- Q1: MFR (none) -> ON Semiconductor; MPN (none) -> BC847CDW1T1G
- U1: MFR (none) -> NXP; MPN (none) -> LPC812M101JDH20
Other:
- note added: "MCU"
- note added: "Power supply"
- moved on the sheet: C3, C4, C6, FB1, J1, U1

Commit message: Swapped SWDCLK and SWDIO - D'oh!
Connections:
- net P2_SWDIO: now also J1.2 (SWDIO/TMS); no longer J1.4 (SWDCLK/TCK)
- net P3_SWCLK: now also J1.4 (SWDCLK/TCK); no longer J1.2 (SWDIO/TMS)
Changed lines of the file:
@@
 Text Label 2500 3700 2    50   ~ 0
 ~RESET
+Text Label 2500 4000 2    50   ~ 0
+P2_SWDIO
 Text Label 2500 3900 2    50   ~ 0
-P2_SWDIO
-Text Label 2500 4000 2    50   ~ 0
 P3_SWCLK
 $Comp
